File: Hardware/VCO/Schematics/VCO-testboard.sch (KiCad schematic (older format))
At the start: 28 parts, among them J1 Conn_01x02, J2 Conn_01x02, J3 Conn_01x02, J4 Conn_01x02, U1 LM358

Commit message: Created VCO testing board
Parts:
- removed unit 1 of U1
- added R8: 10k, Resistors_SMD:R_0805_HandSoldering, symbol R
- C1, C2, C3, C4, C5, C6, C7, C8: footprint (none) -> Capacitors_SMD:C_0805_HandSoldering
- D1, D2, VD1, VD2: footprint (none) -> Diodes_SMD:D_0805
- DA1, U1: footprint (none) -> SMD_Packages:SOIC-8-N
- J1, J2, J3, J4: footprint (none) -> Pin_Headers:Pin_Header_Straight_1x02; symbol Conn_01x02 -> CONN_01X02
- L1: footprint (none) -> Inductors_NEOSID:Neosid_Inductor_Sd8
- R1, R2, R3, R4, R5, R6, R7: footprint (none) -> Resistors_SMD:R_0805_HandSoldering
- R9: renamed from R8; value 110k -> 100k; footprint (none) -> Resistors_SMD:R_0805_HandSoldering
- VT1: footprint (none) -> TO_SOT_Packages_SMD:SOT-23
Connections:
- net +12V: now also U1.8 (V+)
- net GND: now also U1.4 (V-)
- net at R1.2: now also J1.1 (P1)
- net at DA1.2 (-IN), R7.1: now also R8.1; no longer R9.2
- net at DA1.6 (OUT), J4.1 (P1): now also R9.2; no longer R9.1
- net at C6.1, J3.1 (P1), R6.2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: now also U1.1, U1.2 (-); no longer U1.6 (-), U1.7
- net at C2.1, R2.2, R3.1: now also U1.3 (+); no longer U1.5 (+)
- new net: R8.2, R9.1

Commit message: Tuning to avoid 6V source instability and make startup stable
Parts:
- removed C6: 0.1uF, Capacitors_SMD:C_0805_HandSoldering, symbol C
- removed R8: 10k, Resistors_SMD:R_0805_HandSoldering, symbol R
- C3: value 47pF -> 100pF
- L1: value 27 uH -> 22 uH
- R9: value 100k -> 47k
Connections:
- net at DA1.2 (-IN), R7.1: now also R9.1
Other:
- note added: "0V - \nxV - 3.5 MHz\nxV - 3.575 MHz\nxV - 3.65 MHz\n12V -"
Changed lines of the file:
@@
 P 6500 1550
 F 0 "C3" H 6525 1650 50  0000 L CNN
-F 1 "47pF" H 6525 1450 50  0000 L CNN
+F 1 "100pF" H 6525 1450 50  0000 L CNN
 F 2 "Capacitors_SMD:C_0805_HandSoldering" H 6538 1400 50  0001 C CNN
 F 3 "" H 6500 1550 50  0001 C CNN
@@
 P 5600 1975
 F 0 "L1" V 5550 1975 50  0000 C CNN
-F 1 "27 uH" V 5710 1975 50  0000 C CNN
+F 1 "22 uH" V 5710 1975 50  0000 C CNN
 F 2 "Inductors_NEOSID:Neosid_Inductor_Sd8" H 5600 1975 50  0001 C CNN
 F 3 "" H 5600 1975 50  0001 C CNN
@@
 P 9050 2325
 F 0 "R9" V 9130 2325 50  0000 C CNN
-F 1 "100k" V 9050 2325 50  0000 C CNN
+F 1 "47k" V 9050 2325 50  0000 C CNN
 F 2 "Resistors_SMD:R_0805_HandSoldering" V 8980 2325 50  0001 C CNN
 F 3 "" H 9050 2325 50  0001 C CNN
@@
 	7100 3475 8500 3475
 Wire Wire Line
-	7150 3025 7150 3625
-$Comp
-L C C6
-U 1 1 5B78B961
-P 7150 3775
-F 0 "C6" H 7175 3875 50  0000 L CNN
-F 1 "0.1uF" H 7175 3675 50  0000 L CNN
-F 2 "Capacitors_SMD:C_0805_HandSoldering" H 7188 3625 50  0001 C CNN
-F 3 "" H 7150 3775 50  0001 C CNN
-	1    7150 3775
-	1    0    0    -1
-$EndComp
-$Comp
-L GND #PWR018
-U 1 1 5B78B9B8
-P 7150 3975
-F 0 "#PWR018" H 7150 3725 50  0001 C CNN
-F 1 "GND" H 7150 3825 50  0000 C CNN
-F 2 "" H 7150 3975 50  0001 C CNN
-F 3 "" H 7150 3975 50  0001 C CNN
-	1    7150 3975
-	1    0    0    -1
-$EndComp
-Wire Wire Line
 	7500 1650 7500 2000
 Wire Wire Line
@@
 $EndComp
 Wire Wire Line
-	7150 3975 7150 3925
-Wire Wire Line
 	6700 3775 6700 3975
 $Comp
@@
 Wire Wire Line
 	9300 2325 9400 2325
-$Comp
-L R R8
-U 1 1 5BB10FB1
-P 8600 2325
-F 0 "R8" V 8680 2325 50  0000 C CNN
-F 1 "10k" V 8600 2325 50  0000 C CNN
-F 2 "Resistors_SMD:R_0805_HandSoldering" V 8530 2325 50  0001 C CNN
-F 3 "" H 8600 2325 50  0000 C CNN
-	1    8600 2325
-	1    0    0    -1
-$EndComp
-Wire Wire Line
-	8600 2175 8600 2125
+Wire Wire Line
+	8600 2125 8600 2600
 Wire Wire Line
 	8600 2125 8400 2125
 Connection ~ 8400 2125
 Wire Wire Line
-	8600 2475 8600 2600
-Wire Wire Line
 	8600 2600 9050 2600
 Wire Wire Line
@@
 	9050 2125 9300 2125
 Connection ~ 9300 2125
+Wire Wire Line
+	7150 3025 7150 3475
+Text Notes 4250 1400 0    60   ~ 0
+0V - \nxV - 3.5 MHz\nxV - 3.575 MHz\nxV - 3.65 MHz\n12V -
 $EndSCHEMATC

Commit message: VCO is now fully ready
Parts:
- L1: value 22 uH -> 21 uH
Other:
- note added: "0V - 3.115 MHz\n2.8V - 3.5 MHz\n4.3V - 3.575 MHz\n6.3V - 3.65 MHz\n12V - 3.769 MHz"
- note added: "1.7V peak to peak\n3.5MHz"
- note removed: "0V - \nxV - 3.5 MHz\nxV - 3.575 MHz\nxV - 3.65 MHz\n12V -"
- note removed: "1V peak to peak\n3.5MHz"
Changed lines of the file:
@@
 P 5600 1975
 F 0 "L1" V 5550 1975 50  0000 C CNN
-F 1 "22 uH" V 5710 1975 50  0000 C CNN
+F 1 "21 uH" V 5710 1975 50  0000 C CNN
 F 2 "Inductors_NEOSID:Neosid_Inductor_Sd8" H 5600 1975 50  0001 C CNN
 F 3 "" H 5600 1975 50  0001 C CNN
@@
 $EndComp
 Text Notes 9875 2425 0    60   ~ 0
-1V peak to peak\n3.5MHz
+1.7V peak to peak\n3.5MHz
 Text Notes 8800 3550 0    60   ~ 0
 Signal ground - 6V
@@
 	7150 3025 7150 3475
 Text Notes 4250 1400 0    60   ~ 0
-0V - \nxV - 3.5 MHz\nxV - 3.575 MHz\nxV - 3.65 MHz\n12V -
+0V - 3.115 MHz\n2.8V - 3.5 MHz\n4.3V - 3.575 MHz\n6.3V - 3.65 MHz\n12V - 3.769 MHz
 $EndSCHEMATC
