File: Hardware/Prototype 1/Full schematic/Full schematic.sch (KiCad schematic (older format))
At the start: 145 parts, among them J1 Conn_01x04_Male, J4 Conn_01x02_Male, J6 Conn_01x02_Male, J7 Conn_01x02_Male, J8 Conn_01x07_Male, K1 EDR101A0500, K2 EDR101A0500, K3 EDR101A0500, K4 EDR101A0500, K5 EDR101A0500, K6 EDR101A0500, Q1 BSS138, Q2 IRF610, Q3 IRLML2502, Q4 IRLML2502, Q5 IRLML2502, Q6 IRLML2502, Q7 IRLML2502, Q8 IRLML2502, U1 74LVC2T45DC, U2 74LVC2T45DC, U3 AD9835, X1 50MHz

Commit message: Started 144MHz part, have modulated 144MHz carrier
Parts:
- removed C56, C57, C58, C59, C60, C61: 12pF, Capacitor_SMD:C_0805_2012Metric_Pad1.18x1.45mm_HandSolder, symbol Device:C
- removed C? (x6): 0.1uF, symbol Device:C
- removed C?: 470uFx16V, symbol Device:CP
- removed C? (x2): 470uFx6.3V, symbol Device:CP
- removed J8: Conn_01x07_Male, symbol Connector:Conn_01x07_Male
- removed J?: Conn_01x03_Male, symbol Connector:Conn_01x03_Male
- removed J?: Conn_01x04_Male, symbol Connector:Conn_01x04_Male
- removed J?: Conn_01x02_Male, symbol Connector:Conn_01x02_Male
- removed K6: EDR101A0500, Relay_THT:Relay_SPST_StandexMeder_SIL_Form1A, symbol Fossa_library:EDR101A0500
- removed Q8: IRLML2502, Package_TO_SOT_SMD:SOT-23, symbol Device:Q_NMOS_GSD
- removed Q? (x2): BC847, Package_TO_SOT_SMD:SOT-23, symbol Transistor_BJT:BC847
- removed Q?: BSS138, Package_TO_SOT_SMD:SOT-23, symbol Transistor_FET:BSS138
- removed R23: 100, Resistor_SMD:R_0805_2012Metric_Pad1.20x1.40mm_HandSolder, symbol Device:R
- removed R? (x2): 4.7k, symbol Device:R
- removed R? (x2): 30k, symbol Device:R
- removed R? (x2): 6.8k, symbol Device:R
- removed R? (x3): 100, symbol Device:R
- removed R? (x2): 1k, symbol Device:R
- removed R?: 47k, symbol Device:R
- removed R?: 33, symbol Device:R
- removed U?: ICS501, symbol Fossa_library:ICS501
- added C14: 470uF x 16V, Capacitor_THT:CP_Radial_D10.0mm_P5.00mm, symbol Device:CP
- added J2: Conn_01x04_Male, Connector_PinHeader_2.54mm:PinHeader_1x04_P2.54mm_Vertical, symbol Connector:Conn_01x04_Male
- added J3, J5: Conn_01x02_Male, Connector_PinHeader_2.54mm:PinHeader_1x02_P2.54mm_Vertical, symbol Connector:Conn_01x02_Male
- added J8: Conn_01x06_Male, Connector_PinHeader_2.54mm:PinHeader_1x06_P2.54mm_Vertical, symbol Connector:Conn_01x06_Male
- renumbered C19 to C18, C20 to C19, C21 to C20, C22 to C21, C23 to C22, C24 to C23, C25 to C24, C26 to C25, C27 to C26, C28 to C27, C29 to C28, C30 to C29, C31 to C30, C32 to C31, C33 to C32, C34 to C33, C35 to C34, C36 to C35, C37 to C36, C38 to C37, C39 to C38, C40 to C39, C41 to C40, C42 to C41, C43 to C42, C44 to C43, C45 to C44, C46 to C45, C47 to C46, C48 to C47, C49 to C48, C50 to C49, C51 to C50, C52 to C51, C53 to C52, C54 to C53, C55 to C54, C18 to C55
Connections:
- net labels added: +12V
- net labels removed: PWR_144_5, PWR_3.5_12, PWR_3.5_5, PWR_3.5_OUT
- wire segments 369 -> 271
Other:
- note added: "Output stage power"
- note added: "Peak to peak (out):\n3.50MHz - 1V\n3.65MHz - 0.96V\n18.00MHz - 0.8V\n18.25MHz - 0.7V"
- note added: "Power"
- note added: "To ICS501 - 144MHz tract"
- note removed: "144-146MHz 1.5V P-P"
- note removed: "2pF"
- note removed: "3V P-P 18MHz"
- note removed: "Manipulation\nand\nModulation\n1 - OFF\n0 - ON"
- note removed: "PB9"
- note removed: "Peak to peak (out):\n3.50MHz - 1V\n3.65MHz - 0.96V\n18.00MHz - 77mV\n18.25MHz - 77mV"
- note removed: "Power - 3.5MHz"
- note removed: "Power - Common"
- moved on the sheet: C18
