File: Hardware/Full schematic/Full schematic/Full schematic.sch (KiCad schematic (older format))
At the start: 237 parts, among them J1 Conn_01x04_Male, J2 Conn_01x03_Male, J3 Conn_01x02_Male, J4 Conn_01x04_Male, J5 Conn_01x03_Male, J6 Conn_01x02_Male, J7 Conn_01x02_Male, J8 Conn_01x02_Male, J9 Conn_01x07_Male, K1 EDR101A0500, K2 EDR101A0500, K3 EDR101A0500, K4 EDR101A0500, K5 EDR101A0500, K6 EDR101A0500, Q1 BC847, Q10 IRLML2502, Q11 IRLML2502, Q12 IRLML2502, Q13 IRLML2502, Q2 BSS138, Q3 BC847, Q4 IRF610, Q5 BSS138, Q6 BFS17, Q7 AFT05MS003N, Q8 IRLML2502, Q9 IRLML2502, U1 74LVC2T45DC, U2 74LVC2T45DC, U3 AD9835, U4 ICS501, X1 50MHz

Commit message: Support for Bluetooth name and PIN setting
Parts:
- removed C19: 470uFx16V, Capacitor_THT:CP_Radial_D8.0mm_P3.80mm, symbol Device:CP
- removed D? (x3): 1N4148, Diode_THT:D_DO-35_SOD27_P7.62mm_Horizontal, symbol Diode:1N4148
- added C?: 4.7uF, symbol Device:C
- added D? (x7): 1N4148W, Diode_SMD:D_SOD-123, symbol Diode:1N4148W
- added R? (x3): 47k, symbol Device:R
Connections:
- net ENABLE_3.5_VOUT is gone; now on net ENABLE_12V: U?.4 (EN)
- net COMM_5V_ENABLE: now also D?.1 (K), D?.1 (K), D?.1 (K), R?.1
- net DISPLAY_4V: now also D?.2 (A)
- net ENABLE_12V: now also D?.1 (K), R?.1
- net GND: now also C?.2, R?.2, R?.2, R?.2
- net REG_12V: now also C18.1, DA1.7 (+VS), R15.1, C?.1
- net REG_3.3V: now also D?.2 (A)
- net REG_5V: now also D?.2 (A)
- net at C?.2, U?.1 (BOOST): now also D?.1 (K) (x3)
- net DISPLAY_4V_ENABLE renamed ACTIVATE_DISPLAY
- net ACTIVATE_DISPLAY: now also R?.1
- removed net PWR_3.5_12: C18.1, DA1.7 (+VS), J4.3 (Pin_3), R15.1
- new net ACTIVATE_144: D?.2 (A)
- new net ACTIVATE_3.5: D?.2 (A), D?.2 (A)
- new net ACTIVATE_FOX: D?.2 (A)
Other:
- note added: "Power sources activation logic"
Changed lines of the file:
@@
 Wire Wire Line
 	12475 7925 12475 7900
-Text GLabel 11525 1250 1    50   Input ~ 0
-PWR_3.5_12
 Wire Wire Line
 	11250 1350 11525 1350
@@
 Text GLabel 12850 1275 1    50   Input ~ 0
 PWR_3.5_OUT
-$Comp
-L Device:CP C19
-U 1 1 60314788
-P 11025 1500
-F 0 "C19" H 11143 1546 50  0000 L CNN
-F 1 "470uFx16V" H 10825 1400 50  0000 L CNN
-F 2 "Capacitor_THT:CP_Radial_D8.0mm_P3.80mm" H 11063 1350 50  0001 C CNN
-F 3 "~" H 11025 1500 50  0001 C CNN
-	1    11025 1500
-	1    0    0    -1
-$EndComp
-Wire Wire Line
-	11250 1350 11025 1350
 Connection ~ 11250 1350
 $Comp
@@
 Wire Wire Line
 	10800 1675 10800 1650
-Wire Wire Line
-	10800 1350 11025 1350
-Connection ~ 11025 1350
 $Comp
 L power:GND #PWR038
@@
 Wire Wire Line
 	12125 925  12125 900
-Text GLabel 11925 1000 3    50   Input ~ 0
-PWR_3.5_12
-Wire Wire Line
-	11925 1000 11925 900
 Text GLabel 5725 10600 2    50   Input ~ 0
 PWR_3.5_OUT
@@
 Wire Wire Line
 	3350 15425 3350 15400
-$Comp
-L Diode:1N4148 D?
-U 1 1 611FDDCE
-P 3550 14525
-F 0 "D?" H 3550 14742 50  0000 C CNN
-F 1 "1N4148" H 3550 14651 50  0000 C CNN
-F 2 "Diode_THT:D_DO-35_SOD27_P7.62mm_Horizontal" H 3550 14350 50  0001 C CNN
-F 3 "https://assets.nexperia.com/documents/data-sheet/1N4148_1N4448.pdf" H 3550 14525 50  0001 C CNN
-	1    3550 14525
-	1    0    0    -1
-$EndComp
 Wire Wire Line
 	3400 14525 3350 14525
@@
 Wire Wire Line
 	3350 16875 3350 16850
-$Comp
-L Diode:1N4148 D?
-U 1 1 61D4585A
-P 3550 15975
-F 0 "D?" H 3550 16192 50  0000 C CNN
-F 1 "1N4148" H 3550 16101 50  0000 C CNN
-F 2 "Diode_THT:D_DO-35_SOD27_P7.62mm_Horizontal" H 3550 15800 50  0001 C CNN
-F 3 "https://assets.nexperia.com/documents/data-sheet/1N4148_1N4448.pdf" H 3550 15975 50  0001 C CNN
-	1    3550 15975
-	1    0    0    -1
-$EndComp
 Wire Wire Line
 	3400 15975 3350 15975
@@
 Wire Wire Line
 	3350 18400 3350 18375
-$Comp
-L Diode:1N4148 D?
-U 1 1 622ACDA9
-P 3550 17500
-F 0 "D?" H 3550 17717 50  0000 C CNN
-F 1 "1N4148" H 3550 17626 50  0000 C CNN
-F 2 "Diode_THT:D_DO-35_SOD27_P7.62mm_Horizontal" H 3550 17325 50  0001 C CNN
-F 3 "https://assets.nexperia.com/documents/data-sheet/1N4148_1N4448.pdf" H 3550 17500 50  0001 C CNN
-	1    3550 17500
-	1    0    0    -1
-$EndComp
 Wire Wire Line
 	3400 17500 3350 17500
@@
 	2350 17975 2350 17775
 Connection ~ 2350 17775
+Text GLabel 8500 17025 2    50   Input ~ 0
+DISPLAY_4V_ENABLE
+Text GLabel 8500 16825 2    50   Input ~ 0
+COMM_5V_ENABLE
+Text GLabel 8500 16625 2    50   Input ~ 0
+ENABLE_12V
+Text GLabel 8500 16425 2    50   Input ~ 0
+ENABLE_3.5_VOUT
+Text Notes 7425 16250 0    50   ~ 0
+Power sources activation logic
+$Comp
+L Device:R R?
+U 1 1 60C09585
+P 8425 17250
+F 0 "R?" H 8495 17296 50  0000 L CNN
+F 1 "47k" H 8495 17205 50  0000 L CNN
+F 2 "" V 8355 17250 50  0001 C CNN
+F 3 "~" H 8425 17250 50  0001 C CNN
+	1    8425 17250
+	1    0    0    -1
+$EndComp
+$Comp
+L Device:R R?
+U 1 1 60C0A246
+P 8175 17250
+F 0 "R?" H 8245 17296 50  0000 L CNN
+F 1 "47k" H 8245 17205 50  0000 L CNN
+F 2 "" V 8105 17250 50  0001 C CNN
+F 3 "~" H 8175 17250 50  0001 C CNN
+	1    8175 17250
+	1    0    0    -1
+$EndComp
+$Comp
+L Device:R R?
+U 1 1 60C1803F
+P 7925 17250
+F 0 "R?" H 7995 17296 50  0000 L CNN
+F 1 "47k" H 7995 17205 50  0000 L CNN
+F 2 "" V 7855 17250 50  0001 C CNN
+F 3 "~" H 7925 17250 50  0001 C CNN
+	1    7925 17250
+	1    0    0    -1
+$EndComp
+Wire Wire Line
+	8425 17100 8425 17025
+Wire Wire Line
+	8425 17025 8500 17025
+Wire Wire Line
+	8175 17100 8175 16825
+Wire Wire Line
+	8175 16825 8500 16825
+Wire Wire Line
+	7925 17100 7925 16625
+Wire Wire Line
+	7925 16625 8500 16625
+$Comp
+L power:GND #PWR?
+U 1 1 60EE6215
+P 7925 17425
+F 0 "#PWR?" H 7925 17175 50  0001 C CNN
+F 1 "GND" H 7930 17252 50  0000 C CNN
+F 2 "" H 7925 17425 50  0001 C CNN
+F 3 "" H 7925 17425 50  0001 C CNN
+	1    7925 17425
+	1    0    0    -1
+$EndComp
+$Comp
+L power:GND #PWR?
+U 1 1 60EE7333
+P 8175 17425
+F 0 "#PWR?" H 8175 17175 50  0001 C CNN
+F 1 "GND" H 8180 17252 50  0000 C CNN
+F 2 "" H 8175 17425 50  0001 C CNN
+F 3 "" H 8175 17425 50  0001 C CNN
+	1    8175 17425
+	1    0    0    -1
+$EndComp
+$Comp
+L power:GND #PWR?
+U 1 1 60EE83A0
+P 8425 17425
+F 0 "#PWR?" H 8425 17175 50  0001 C CNN
+F 1 "GND" H 8430 17252 50  0000 C CNN
+F 2 "" H 8425 17425 50  0001 C CNN
+F 3 "" H 8425 17425 50  0001 C CNN
+	1    8425 17425
+	1    0    0    -1
+$EndComp
+Wire Wire Line
+	7925 17425 7925 17400
+Wire Wire Line
+	8175 17425 8175 17400
+Wire Wire Line
+	8425 17425 8425 17400
+Text GLabel 7075 16825 0    50   Input ~ 0
+ACTIVATE_FOX
+Text GLabel 7300 16425 0    50   Input ~ 0
+ACTIVATE_3.5
+Text GLabel 7075 17025 0    50   Input ~ 0
+ACTIVATE_144
+$Comp
+L Diode:1N4148W D?
+U 1 1 61261C07
+P 7275 16825
+F 0 "D?" H 7275 16608 50  0000 C CNN
+F 1 "1N4148W" H 7275 16699 50  0000 C CNN
+F 2 "Diode_SMD:D_SOD-123" H 7275 16650 50  0001 C CNN
+F 3 "https://www.vishay.com/docs/85748/1n4148w.pdf" H 7275 16825 50  0001 C CNN
+	1    7275 16825
+	-1   0    0    1
+$EndComp
+$Comp
+L Diode:1N4148W D?
+U 1 1 6126CF80
+P 3550 17500
+F 0 "D?" H 3550 17717 50  0000 C CNN
+F 1 "1N4148W" H 3550 17626 50  0000 C CNN
+F 2 "Diode_SMD:D_SOD-123" H 3550 17325 50  0001 C CNN
+F 3 "https://www.vishay.com/docs/85748/1n4148w.pdf" H 3550 17500 50  0001 C CNN
+	1    3550 17500
+	1    0    0    -1
+$EndComp
+$Comp
+L Diode:1N4148W D?
+U 1 1 61301B9C
+P 3550 15975
+F 0 "D?" H 3550 16192 50  0000 C CNN
+F 1 "1N4148W" H 3550 16101 50  0000 C CNN
+F 2 "Diode_SMD:D_SOD-123" H 3550 15800 50  0001 C CNN
+F 3 "https://www.vishay.com/docs/85748/1n4148w.pdf" H 3550 15975 50  0001 C CNN
+	1    3550 15975
+	1    0    0    -1
+$EndComp
+$Comp
+L Diode:1N4148W D?
+U 1 1 613967DF
+P 3550 14525
+F 0 "D?" H 3550 14742 50  0000 C CNN
+F 1 "1N4148W" H 3550 14651 50  0000 C CNN
+F 2 "Diode_SMD:D_SOD-123" H 3550 14350 50  0001 C CNN
+F 3 "https://www.vishay.com/docs/85748/1n4148w.pdf" H 3550 14525 50  0001 C CNN
+	1    3550 14525
+	1    0    0    -1
+$EndComp
+$Comp
+L Diode:1N4148W D?
+U 1 1 616883CD
+P 7700 16425
+F 0 "D?" H 7725 16525 50  0000 C CNN
+F 1 "1N4148W" H 7700 16350 50  0000 C CNN
+F 2 "Diode_SMD:D_SOD-123" H 7700 16250 50  0001 C CNN
+F 3 "https://www.vishay.com/docs/85748/1n4148w.pdf" H 7700 16425 50  0001 C CNN
+	1    7700 16425
+	-1   0    0    1
+$EndComp
+$Comp
+L Diode:1N4148W D?
+U 1 1 617B14AE
+P 7500 16600
+F 0 "D?" H 7500 16817 50  0000 C CNN
+F 1 "1N4148W" H 7500 16726 50  0000 C CNN
+F 2 "Diode_SMD:D_SOD-123" H 7500 16425 50  0001 C CNN
+F 3 "https://www.vishay.com/docs/85748/1n4148w.pdf" H 7500 16600 50  0001 C CNN
+	1    7500 16600
+	0    -1   -1   0
+$EndComp
+Wire Wire Line
+	7925 16625 7925 16425
+Connection ~ 7925 16625
+Wire Wire Line
+	7925 16425 8500 16425
+Wire Wire Line
+	7850 16425 7925 16425
+Connection ~ 7925 16425
+Wire Wire Line
+	7550 16425 7500 16425
+Wire Wire Line
+	7500 16425 7500 16450
+Wire Wire Line
+	8175 16825 7500 16825
+Wire Wire Line
+	7500 16825 7500 16750
+Connection ~ 8175 16825
+Wire Wire Line
+	7300 16425 7500 16425
+Connection ~ 7500 16425
+Wire Wire Line
+	7425 16825 7500 16825
+Connection ~ 7500 16825
+Wire Wire Line
+	7125 16825 7075 16825
+$Comp
+L Diode:1N4148W D?
+U 1 1 61FD5871
+P 7275 17025
+F 0 "D?" H 7275 16808 50  0000 C CNN
+F 1 "1N4148W" H 7275 16899 50  0000 C CNN
+F 2 "Diode_SMD:D_SOD-123" H 7275 16850 50  0001 C CNN
+F 3 "https://www.vishay.com/docs/85748/1n4148w.pdf" H 7275 17025 50  0001 C CNN
+	1    7275 17025
+	-1   0    0    1
+$EndComp
+Text GLabel 7525 17150 0    50   Input ~ 0
+ACTIVATE_DISPLAY
+Wire Wire Line
+	7075 17025 7125 17025
+Wire Wire Line
+	7425 17025 7500 17025
+Wire Wire Line
+	7500 16825 7500 17025
+Wire Wire Line
+	7525 17150 7600 17150
+Wire Wire Line
+	7600 17150 7600 17025
+Wire Wire Line
+	7600 17025 8425 17025
+Connection ~ 8425 17025
+Text GLabel 11525 1250 1    50   Input ~ 0
+REG_12V
+Wire Wire Line
+	10800 1350 11025 1350
+$Comp
+L Device:C C?
+U 1 1 624CD754
+P 11025 1500
+F 0 "C?" H 11140 1546 50  0000 L CNN
+F 1 "4.7uF" H 11140 1455 50  0000 L CNN
+F 2 "" H 11063 1350 50  0001 C CNN
+F 3 "~" H 11025 1500 50  0001 C CNN
+	1    11025 1500
+	1    0    0    -1
+$EndComp
+Connection ~ 11025 1350
+Wire Wire Line
+	11025 1350 11250 1350
 $EndSCHEMATC
