File: Hardware/Full schematic/Full schematic/Full schematic.kicad_pcb (KiCad board)
At the start: 2 copper layers, 329 parts, among them J1 Conn_01x02_Male, J10 Conn_01x01_Male, J2 Reset, J3 Encoder, J4 Failure LED, J5 Bluetooth, J6 Conn_01x02_Male, J7 Display, J8 Buttons, J9 Conn_01x02_Male, K1 EDR101A0500, K2 EDR101A0500, K3 EDR101A0500, K4 EDR101A0500, K5 EDR101A0500, K6 EDR101A0500, Q1 BC847, Q10 IRLML6402, Q11 BC847, Q12 IRFZ44, Q13 BC847, Q14 BSS138, Q15 BC847, Q16 IRF610, Q17 BC847, Q18 IRLML6402, Q19 BC847, Q2 BC847, Q20 BFS17, Q21 IRLML6402, Q22 AFT05MS003N, Q23 IRLML2502, Q24 IRLML2502, Q25 IRLML2502, Q26 IRLML2502, Q27 IRLML2502, Q28 IRLML2502, Q3 BC847, Q4 BC847, Q5 BC847, Q6 IRLML6402, Q7 IRF4905, Q8 IRLML6402, Q9 IRLML6402, U1 74LVC2T45DC, U10 ICS501, U11 STM32F103C8Tx, U12 CAT24C256, U2 74LVC2T45DC, U3 AD9835, U4 LM27313XMF, U5 LM2734X, U6 LM2734X, U7 LM2734X, U8 UC3843_SOIC8, U9 AD5245BRJZ10, X1 50MHz, Y1 8MHz, Y2 32768Hz

Commit message: PCB tracing in progress
Parts:
- J6, L12, Q16, RV1: moved to B.Cu
- L11: footprint Inductor_THT:L_Radial_D9.5mm_P5.00mm_Fastron_07HVP -> Inductor_SMD:L_1812_4532Metric_Pad1.30x3.40mm_HandSolder
- moved L12 145.4 mm to (185.4, 113.3), turned to 270 degrees
- moved L11 113.9 mm to (181.9, 100.4), turned to 90 degrees
- moved J6 102.1 mm to (188.7, 127.3), turned to 90 degrees
- moved Q16 102.0 mm to (191.8, 100.6), turned to 180 degrees
- moved DA1 101.0 mm to (178.2, 110.9)
- moved RV1 93.7 mm to (173.2, 114.0)
- moved C72 77.8 mm to (186.7, 115.8)
- moved C59 77.2 mm to (178.0, 107.2), turned to 180 degrees
- moved C69 76.4 mm to (188.2, 113.3)
- moved C67 76.1 mm to (182.1, 106.7)
- moved C60 71.2 mm to (178.0, 105.2), turned to 180 degrees
- moved R63 66.4 mm to (176.3, 114.6), turned to 180 degrees
- moved C68 64.3 mm to (182.1, 104.6)
- moved C56 61.1 mm to (170.7, 111.5), turned to 180 degrees
- moved C63 56.9 mm to (174.3, 105.2)
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Routing:
- net GND: track 404.5 -> 473.2 mm, vias 4 -> 8
- net ANT_3.5: track 31.2 -> 66.0 mm
- net Net-(C69-Pad2): track 0.00 -> 22.3 mm
- net Net-(DA1-Pad6): track 0.00 -> 21.4 mm, vias 0 -> 1
- net PWR_3.5_12: track 65.8 -> 77.5 mm, vias 4 -> 6
- net Net-(DA1-Pad2): track 0.00 -> 7.62 mm
- net Net-(C63-Pad1): track 0.00 -> 6.51 mm
- net Net-(Q14-Pad1): track 0.00 -> 5.59 mm
- net PWR_3.5_5: track 40.2 -> 45.0 mm
- net PWR_3.5_OUT: track 11.2 -> 15.6 mm
- net Net-(C69-Pad1): track 0.00 -> 4.37 mm
- net Net-(C56-Pad1): track 0.00 -> 4.04 mm

Commit message: PCB tracing in progress
Parts:
- C110, C75, J9, L13, L14, L15, RV2: moved to B.Cu
- moved L13 175.0 mm to (218.3, 134.2), turned to 270 degrees
- moved L14 171.8 mm to (229.7, 151.0), turned to 90 degrees
- moved L15 158.3 mm to (231.3, 136.1), turned to 90 degrees
- moved C110 154.7 mm to (221.1, 146.4)
- moved U10 145.0 mm to (209.4, 144.8)
- moved RV2 144.5 mm to (222.4, 135.5), turned to 180 degrees
- moved Q22 140.1 mm to (226.4, 139.4), turned to 90 degrees
- moved C96 130.2 mm to (222.3, 150.1)
- moved J9 127.2 mm to (227.2, 132.3)
- moved C74 126.0 mm to (216.0, 137.3)
- moved C97 124.5 mm to (231.0, 141.5), turned to 180 degrees
- moved C99 122.6 mm to (222.3, 148.2)
- moved C75 120.4 mm to (212.2, 135.5)
- moved C71 118.4 mm to (216.0, 139.2)
- moved C77 117.6 mm to (215.1, 145.8), turned to 270 degrees
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Routing:
- net GND: track 473.2 -> 586.8 mm, vias 8 -> 13
- net PWR_144_5: track 0.00 -> 57.4 mm, vias 0 -> 1
- net PWR_144_OUT: track 0.00 -> 13.7 mm
- net Net-(C84-Pad1): track 0.00 -> 10.3 mm, vias 0 -> 1
- net Net-(C61-Pad1): track 0.00 -> 9.78 mm
- net Net-(C54-Pad2): track 0.00 -> 9.20 mm
- net Net-(C113-Pad1): track 0.00 -> 8.88 mm
- net Net-(C77-Pad1): track 0.00 -> 6.76 mm
- net MANIP_144: track 0.00 -> 6.63 mm
- net Net-(C65-Pad1): track 0.00 -> 6.55 mm
- net Net-(C65-Pad2): track 0.00 -> 5.74 mm
- net Net-(C101-Pad1): track 0.00 -> 5.65 mm
- net Net-(C84-Pad2): track 0.00 -> 5.45 mm
- net Net-(C61-Pad2): track 0.00 -> 5.30 mm
- net Net-(Q19-Pad3): track 0.00 -> 4.90 mm
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
Commit message: PCB tracing in progress
Parts:
- C18, C2, C3, C7, C8, X1: moved to B.Cu
- moved X1 139.4 mm to (184.9, 143.0), turned to 270 degrees
- moved L9 118.9 mm to (176.9, 118.1)
- moved C7 114.8 mm to (180.5, 146.4)
- moved U3 111.1 mm to (181.5, 138.0), turned to 90 degrees
- moved U1 109.7 mm to (190.5, 140.2), turned to 180 degrees
- moved R33 108.2 mm to (180.5, 144.5), turned to 180 degrees
- moved C4 107.7 mm to (190.5, 142.5)
- moved U2 101.8 mm to (190.5, 134.0), turned to 180 degrees
- moved C5 100.2 mm to (190.5, 136.3)
- moved C24 100.2 mm to (181.0, 130.5), turned to 270 degrees
- moved C3 99.9 mm to (190.5, 131.7)
- moved R1 98.7 mm to (194.7, 141.2)
- moved C18 98.4 mm to (181.5, 137.0)
- moved C2 97.9 mm to (190.5, 138.0)
- moved L2 95.6 mm to (176.9, 130.3), turned to 180 degrees
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Routing:
- net GND: track 586.8 -> 651.6 mm, vias 13 -> 19
- net Net-(C54-Pad1): track 0.00 -> 51.8 mm
- net REG_5V: track 44.0 -> 73.9 mm, vias 1 -> 3
- net REG_3.3V: track 63.7 -> 83.9 mm, vias 1 -> 7
- net Net-(C36-Pad1): track 0.00 -> 12.4 mm, vias 0 -> 2
- net Net-(U3-Pad6): track 0.00 -> 11.8 mm
- net Net-(C44-Pad1): track 0.00 -> 10.9 mm, vias 0 -> 2
- net Net-(C31-Pad1): track 0.00 -> 8.40 mm
- net Net-(R33-Pad2): track 0.00 -> 4.83 mm
- net Net-(R26-Pad2): track 0.00 -> 4.15 mm
- net Net-(C24-Pad2): track 0.00 -> 3.77 mm
- net Net-(R27-Pad1): track 0.00 -> 3.37 mm
- net Net-(R26-Pad1): track 0.00 -> 2.92 mm
- net Net-(R25-Pad1): track 0.00 -> 2.61 mm
- net Net-(C22-Pad1): track 0.00 -> 2.50 mm
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
Commit message: PCB tracing in progress
Parts:
- C108, C109, C76, C78, C81, C85, C86, C94, C98, J2, J3, J4, J5, J7, J8, JP1, JP2, JP3, JP4, R88, R90, R91, R92, Y1, Y2: moved to B.Cu
- moved R88 194.4 mm to (136.8, 221.9), turned to 90 degrees
- moved J3 185.1 mm to (157.0, 211.7), turned to 270 degrees
- moved C70 183.5 mm to (127.5, 217.7), turned to 180 degrees
- moved C93 178.9 mm to (136.8, 221.9), turned to 270 degrees
- moved R5 178.3 mm to (62.6, 178.1)
- moved C108 168.5 mm to (143.0, 223.8), turned to 180 degrees
- moved C82 167.4 mm to (133.7, 205.3), turned to 90 degrees
- moved J5 167.2 mm to (160.4, 208.2), turned to 90 degrees
- moved C86 165.0 mm to (142.5, 209.8)
- moved U12 162.1 mm to (143.8, 222.0), turned to 90 degrees
- moved J4 159.4 mm to (136.3, 206.2)
- moved U11 157.8 mm to (142.4, 209.3)
- moved J7 156.8 mm to (155.7, 200.2), turned to 90 degrees
- moved R78 154.4 mm to (162.1, 214.4), turned to 90 degrees
- moved J8 154.4 mm to (134.2, 219.2), turned to 270 degrees
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Routing:
- net GND: track 651.6 -> 806.9 mm, vias 19 -> 27
- net REG_3.3V: track 83.9 -> 192.4 mm, vias 7 -> 14
- net ENABLE_BT: track 0.00 -> 70.7 mm, vias 0 -> 2
- net ENCODER_BTN: track 0.00 -> 21.9 mm
- net ENCODER_R: track 0.00 -> 19.1 mm
- net SWDIO: track 0.00 -> 18.6 mm
- net RESET: track 0.00 -> 16.5 mm
- net Net-(C79-Pad1): track 0.00 -> 14.6 mm
- net ENCODER_L: track 0.00 -> 14.5 mm
- net BOOT1: track 0.00 -> 14.0 mm, vias 0 -> 1
- net Net-(C80-Pad1): track 0.00 -> 13.5 mm
- net DISPLAY_SCL: track 0.00 -> 13.5 mm
- net BTN_LEFT: track 0.00 -> 12.6 mm
- net BTN_RIGHT: track 0.00 -> 12.1 mm
- net DISPLAY_SDA: track 0.00 -> 11.6 mm
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
Commit message: PCB tracing in progress
Parts:
- C100: moved to B.Cu
- moved D1 137.2 mm to (59.6, 180.3), turned to 270 degrees
- moved R7 129.6 mm to (85.2, 156.7), turned to 90 degrees
- moved R18 122.9 mm to (87.0, 153.8), turned to 180 degrees
- moved Q6 115.3 mm to (90.6, 156.7)
- moved C6 110.8 mm to (92.3, 151.8), turned to 180 degrees
- moved C100 110.6 mm to (145.3, 209.0), turned to 270 degrees
- moved R23 109.9 mm to (93.2, 156.7), turned to 90 degrees
- moved R10 109.4 mm to (197.6, 147.3), turned to 180 degrees
- moved D2 107.0 mm to (57.1, 180.3), turned to 270 degrees
- moved D3 101.8 mm to (54.7, 180.3), turned to 270 degrees
- moved R22 100.2 mm to (201.3, 143.9), turned to 180 degrees
- moved Q1 97.5 mm to (83.4, 153.2)
- moved R6 90.5 mm to (83.5, 150.4)
- moved R11 81.8 mm to (197.6, 149.2)
- moved Q5 73.5 mm to (197.6, 144.6), turned to 180 degrees
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Routing:
- net ACTIVATE_3.5: track 0.00 -> 79.9 mm, vias 1 -> 2
- net GND: track 806.9 -> 837.0 mm
- net REG_5V: track 77.0 -> 92.9 mm, vias 3 -> 5
- net BATT_7.4V: track 86.2 -> 96.2 mm, vias 0 -> 1
- net COMM_5V_ENABLE: track 4.67 -> 11.8 mm
- net DDS_SDATA: track 0.00 -> 7.13 mm, vias 0 -> 1
- net REG_3.3V: track 192.4 -> 197.3 mm, vias 14 -> 15
- net ADC_UBATT: track 0.00 -> 3.99 mm
- net Net-(Q5-Pad3): track 0.00 -> 3.96 mm
- net Net-(Q6-Pad1): track 0.00 -> 3.66 mm
- net DDS_SCLK: track 2.36 -> 5.39 mm, vias 1 -> 2
- net Net-(Q6-Pad3): track 0.00 -> 2.06 mm
- net Net-(Q10-Pad1): track 1.69 -> 3.69 mm
- net ACTIVATE_144: track 0.00 -> 1.91 mm
- net Net-(Q1-Pad1): track 0.00 -> 1.89 mm
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
Commit message: PCB tracing in progress - almost done
Parts:
- J10: moved to B.Cu
- moved R4 135.2 mm to (77.4, 173.6), turned to 180 degrees
- moved R67 110.8 mm to (86.4, 148.6), turned to 270 degrees
- moved R21 110.5 mm to (213.8, 150.7), turned to 180 degrees
- moved R15 109.4 mm to (216.6, 151.8), turned to 90 degrees
- moved R9 99.8 mm to (207.5, 150.8), turned to 270 degrees
- moved J10 98.6 mm to (109.9, 141.7), turned to 90 degrees
- moved Q9 97.4 mm to (219.3, 151.7)
- moved Q17 95.3 mm to (120.7, 133.1), turned to 180 degrees
- moved R74 94.5 mm to (118.0, 133.0), turned to 90 degrees
- moved R69 93.9 mm to (116.3, 133.0), turned to 270 degrees
- moved Q18 93.2 mm to (113.9, 133.1), turned to 180 degrees
- moved R68 90.9 mm to (120.7, 136.3), turned to 0 degrees
- moved Q4 89.1 mm to (210.2, 150.7)
- moved JP3 87.1 mm to (110.3, 137.0), turned to 0 degrees
- moved C76 86.5 mm to (119.3, 139.1), turned to 0 degrees
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Routing:
- net GND: track 837.0 -> 859.2 mm, vias 27 -> 28
- net ACTIVATE_144: track 1.91 -> 13.9 mm
- net Net-(Q9-Pad1): track 0.00 -> 3.52 mm
- net PWR_3.5_OUT: track 15.6 -> 17.6 mm
- net ADC_U3.5_OUT: track 0.00 -> 1.87 mm
- net BATT_7.4V: track 96.2 -> 98.0 mm
- net Net-(Q4-Pad1): track 0.00 -> 1.71 mm
- net Net-(Q4-Pad3): track 0.00 -> 1.56 mm
- net PWR_144_OUT: track 13.7 -> 14.8 mm
- net ACTIVATE_3.5: vias 2 -> 1

Commit message: PCB tracing in progress
Parts:
- moved R90 3.76 mm to (127.2, 155.2)
- moved U12 3.76 mm to (129.2, 154.4)
- moved R92 3.76 mm to (129.1, 155.2)
- moved C108 3.76 mm to (131.0, 155.2)
- moved J8 3.76 mm to (126.4, 164.0)
- moved R88 3.76 mm to (129.1, 161.4)
- moved C93 3.76 mm to (129.1, 161.4)
- moved C95 3.76 mm to (129.1, 164.0)
- moved R91 3.76 mm to (129.1, 164.0)
Routing:
- net ACTIVATE_DISPLAY: track 2.16 -> 188.1 mm, vias 2 -> 3
- net ACTIVATE_FOX: track 0.00 -> 167.9 mm, vias 0 -> 2
- net ACTIVATE_144: track 13.9 -> 174.4 mm, vias 0 -> 2
- net ADC_U3.5_OUT: track 1.87 -> 81.9 mm, vias 0 -> 2
- net ADC_UBATT: track 3.99 -> 69.8 mm, vias 0 -> 2
- net DISPLAY_4V: track 24.2 -> 61.6 mm, vias 0 -> 3
- net ENABLE_UBATT_CHECK: track 0.00 -> 34.7 mm, vias 1 -> 2
- net ACTIVATE_3.5: track 79.9 -> 111.7 mm, vias 1 -> 7
- net ENABLE_BT: track 70.7 -> 44.3 mm
- net GND: track 859.2 -> 881.3 mm
- net REG_3.3V: track 197.3 -> 208.4 mm, vias 15 -> 16
- net DDS_SDATA: track 7.13 -> 12.6 mm, vias 1 -> 2
- net I2C2_SCL: track 6.99 -> 11.7 mm
- net I2C2_SDA: track 10.3 -> 14.7 mm
- net MATCH_5: track 0.00 -> 4.26 mm, vias 1 -> 2
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
Commit message: PCB tracing in progress - need to connect transmitters unit
Parts:
- moved C78 4.25 mm to (115.0, 141.7)
- moved C79 4.25 mm to (106.7, 175.1)
- moved C81 4.25 mm to (115.0, 144.3)
- moved C82 4.25 mm to (106.0, 167.5)
- moved C86 4.25 mm to (110.5, 158.7)
- moved C94 4.25 mm to (108.5, 158.8)
- moved J10 4.25 mm to (105.6, 141.7)
- moved J2 4.25 mm to (116.0, 172.3)
- moved J3 4.25 mm to (112.4, 144.3)
- moved J4 4.25 mm to (106.9, 165.0)
- moved J7 4.25 mm to (100.8, 145.5)
- moved JP1 4.25 mm to (100.8, 161.8)
- moved Q17 4.25 mm to (116.5, 133.2)
- moved R68 4.25 mm to (116.4, 136.4)
- moved R69 4.25 mm to (112.0, 133.1)
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Routing:
- net I2C2_SDA: track 14.7 -> 98.3 mm, vias 1 -> 4
- net I2C2_SCL: track 11.7 -> 91.8 mm, vias 1 -> 4
- net REG_5V: track 92.9 -> 170.2 mm, vias 5 -> 8
- net ACTIVATE_3.5: track 111.7 -> 89.9 mm
- net ACTIVATE_DISPLAY: track 188.1 -> 183.8 mm
- net ADC_UBATT: track 69.8 -> 65.6 mm
- net ENABLE_UBATT_CHECK: track 34.7 -> 30.4 mm
- net ADC_U3.5_OUT: track 81.9 -> 77.6 mm
- net ACTIVATE_FOX: track 167.9 -> 163.6 mm
- net ACTIVATE_144: track 174.4 -> 170.2 mm
- net REG_3.3V: track 208.4 -> 204.2 mm
- net GND: track 881.3 -> 877.1 mm
- net DISPLAY_4V: track 61.6 -> 58.2 mm
