File: Hardware/Schematic v1/Full schematic/Full schematic.kicad_pcb (KiCad board)
At the start: 2 copper layers, 120 x 48.3 mm, 303 parts, among them J1 Conn_01x02_Male, J10 Conn_01x03_Male, J2 Reset, J3 Encoder, J4 Failure LED, J5 Bluetooth, J6 Conn_01x02_Male, J7 Display, J8 Buttons, J9 Conn_01x02_Male, K1 IM43TS, K2 IM43TS, K3 IM43TS, K4 IM43TS, K5 IM43TS, K6 IM43TS, Q1 BC847, Q10 IRLML6402, Q11 BC847, Q12 IRFZ44, Q13 BC847, Q14 IRLML6402, Q15 BC847, Q16 BSS138, Q17 BC847, Q18 IRF610, Q19 BC847, Q2 BC847, Q20 IRLML6402, Q21 BC847, Q22 IRLML6402, Q23 BFS17, Q24 AFT05MS003N, Q3 BC847, Q4 BC847, Q5 BC847, Q6 IRLML6402, Q7 IRF4905, Q8 IRLML6402, Q9 IRLML6402, U1 74LVC2T45DC, U10 ICS501, U11 STM32F103C8Tx, U12 MCP23017_SS, U13 CAT24C256, U2 74LVC2T45DC, U3 AD9835, U4 LM27313XMF, U5 LM2734X, U6 LM2734X, U7 MAX1837EUT33-T, U8 UC3843_SOIC8, U9 AD5245BRJZ10, X1 50MHz, Y1 8MHz, Y2 32768Hz

Commit message: - PCB tracing in progress
Parts:
- C59, C60, C73, C85, C89, C92, C96, J9, L13, L14, L15, Q15, Q17, Q21, R53, R63, R66, R82, R87, R91, RV2, U10: moved to B.Cu
- moved L13 268.2 mm to (347.7, 71.0), turned to -90 degrees
- moved Q24 267.2 mm to (343.7, 82.5), turned to 180 degrees
- moved L14 261.5 mm to (344.0, 81.7), turned to 90 degrees
- moved R88 252.0 mm to (350.0, 69.3)
- moved Q23 251.2 mm to (345.1, 74.1), turned to 90 degrees
- moved C89 241.6 mm to (348.1, 86.3), turned to 90 degrees
- moved C90 237.2 mm to (347.5, 80.5), turned to 180 degrees
- moved U10 233.9 mm to (335.0, 76.2)
- moved C68 226.3 mm to (335.2, 76.3)
- moved R85 223.3 mm to (344.0, 77.0)
- moved C92 221.6 mm to (350.0, 86.3), turned to 90 degrees
- moved R82 219.9 mm to (345.3, 70.1), turned to 90 degrees
- moved RV2 218.3 mm to (351.0, 70.9), turned to 180 degrees
- moved C96 215.6 mm to (336.3, 87.3), turned to 90 degrees
- moved J9 213.9 mm to (353.9, 82.8)
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Routing:
- net GND: track 121.8 -> 208.0 mm, vias 5 -> 21
- net PWR_144_5: track 0.00 -> 56.9 mm, vias 0 -> 3
- net Manipulation: track 0.00 -> 35.6 mm, vias 0 -> 5
- net Net-(C60-Pad1): track 0.00 -> 14.2 mm, vias 0 -> 1
- net PWR_144_OUT: track 0.00 -> 13.7 mm
- net Net-(C82-Pad1): track 0.00 -> 13.7 mm, vias 0 -> 1
- net Net-(C75-Pad2): track 0.00 -> 6.93 mm, vias 0 -> 1
- net Net-(C75-Pad1): track 0.00 -> 5.85 mm
- net Net-(R71-Pad2): track 0.00 -> 4.96 mm, vias 0 -> 1
- net Net-(C85-Pad1): track 0.00 -> 4.91 mm, vias 0 -> 1
- net Net-(Q21-Pad3): track 0.00 -> 4.24 mm
- net Net-(C82-Pad2): track 0.00 -> 4.23 mm, vias 0 -> 1
- net Net-(C59-Pad2): track 0.00 -> 4.05 mm, vias 0 -> 1
- net Net-(C52-Pad2): track 0.00 -> 3.95 mm, vias 0 -> 2
- net Net-(C63-Pad1): track 0.00 -> 3.85 mm, vias 0 -> 1
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
Commit message: RF parts and frequency synthesizer traced
Parts:
- C2, C23, C29, C3, C36, C4, C41, C5, L2, L6, L7, L9, X1: moved to B.Cu
- moved U2 233.7 mm to (315.0, 76.2), turned to -90 degrees
- moved X1 232.2 mm to (306.5, 85.6), turned to 180 degrees
- moved L2 226.1 mm to (311.3, 84.0), turned to -90 degrees
- moved U1 208.1 mm to (311.0, 73.9), turned to -90 degrees
- moved C29 203.4 mm to (315.2, 80.0)
- moved C5 198.6 mm to (315.8, 76.2), turned to 90 degrees
- moved C8 196.0 mm to (310.5, 81.9), turned to -90 degrees
- moved R47 190.8 mm to (325.4, 81.0), turned to 90 degrees
- moved C2 190.4 mm to (310.1, 73.9), turned to 90 degrees
- moved U3 181.8 mm to (315.2, 82.7)
- moved C41 181.6 mm to (323.1, 80.0)
- moved L7 177.3 mm to (319.2, 84.0), turned to -90 degrees
- moved C36 176.9 mm to (319.2, 80.0)
- moved C4 175.8 mm to (311.9, 73.9), turned to 90 degrees
- moved C7 174.0 mm to (302.7, 81.9), turned to 180 degrees
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Routing:
- net GND: track 208.0 -> 282.0 mm, vias 21 -> 29
- net Net-(C52-Pad1): track 0.00 -> 45.3 mm, vias 0 -> 6
- net REG_5V: track 0.00 -> 44.3 mm, vias 0 -> 4
- net Net-(U3-Pad6): track 0.00 -> 29.6 mm
- net Net-(R26-Pad2): track 0.00 -> 26.1 mm, vias 0 -> 2
- net SW_3.3V: track 0.00 -> 13.6 mm, vias 0 -> 2
- net Net-(R28-Pad2): track 0.00 -> 13.0 mm, vias 0 -> 2
- net Net-(C23-Pad2): track 0.00 -> 12.9 mm, vias 0 -> 1
- net Net-(C22-Pad1): track 0.00 -> 12.3 mm
- net Net-(R27-Pad2): track 0.00 -> 12.1 mm, vias 0 -> 2
- net Net-(C36-Pad1): track 0.00 -> 10.8 mm
- net Net-(C29-Pad1): track 0.00 -> 8.76 mm
- net Net-(C41-Pad1): track 0.00 -> 8.28 mm
- net Net-(R2-Pad1): track 0.00 -> 6.89 mm
- net Net-(R1-Pad1): track 0.00 -> 6.81 mm
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
Commit message: PCB tracing in progress
Parts:
- C1: footprint Inductor_SMD:L_0603_1608Metric_Pad1.05x0.95mm_HandSolder -> Capacitor_THT:CP_Radial_D6.3mm_P2.50mm; moved to B.Cu
- C10, C12, C17, C20, C24, C28, C31, C37, C38, C40, C47, C48, C51, C57, C62, C9, D10, D11, J1, L1, L3, L4, Q12, Q7, R29, R31, R35, R38, R44, R45, R46, R48, R58: moved to B.Cu
- moved Q12 227.0 mm to (276.9, 54.6), turned to 180 degrees
- moved C51 221.3 mm to (278.4, 49.9), turned to 90 degrees
- moved C55 214.0 mm to (294.6, 47.1), turned to 90 degrees
- moved U9 213.8 mm to (291.3, 56.8)
- moved L10 213.6 mm to (286.8, 48.4)
- moved R46 208.4 mm to (261.5, 58.5), turned to 90 degrees
- moved C49 196.0 mm to (279.3, 47.3), turned to 90 degrees
- moved C57 188.8 mm to (294.9, 49.7), turned to 90 degrees
- moved C40 187.5 mm to (249.1, 60.6), turned to 180 degrees
- moved Q2 186.9 mm to (249.0, 47.0), turned to -90 degrees
- moved D10 185.1 mm to (278.8, 57.0)
- moved J1 183.9 mm to (238.1, 51.7)
- moved R57 183.3 mm to (294.4, 52.4), turned to -90 degrees
- moved C28 180.4 mm to (254.0, 49.9), turned to 90 degrees
- moved C48 180.3 mm to (254.9, 67.3), turned to 90 degrees
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Routing:
- net GND: track 282.0 -> 479.7 mm, vias 29 -> 35
- net BATT_7.4V: track 0.00 -> 41.9 mm
- net Net-(C19-Pad2): track 0.00 -> 36.3 mm, vias 0 -> 2
- net POWERS_3.5: track 0.00 -> 25.9 mm, vias 0 -> 2
- net REG_5V: track 44.3 -> 66.6 mm, vias 4 -> 6
- net Net-(D11-Pad2): track 0.00 -> 20.0 mm
- net Net-(Q12-Pad3): track 0.00 -> 16.7 mm
- net Net-(Q11-Pad2): track 0.00 -> 15.9 mm, vias 0 -> 2
- net Net-(C49-Pad1): track 0.00 -> 13.3 mm
- net Net-(C13-Pad1): track 0.00 -> 12.4 mm
- net DISPLAY_4V: track 0.00 -> 11.9 mm, vias 0 -> 2
- net PWR_3.5_OUT: track 4.17 -> 14.7 mm
- net Net-(C26-Pad1): track 0.00 -> 7.27 mm, vias 0 -> 1
- net Net-(C27-Pad1): track 0.00 -> 7.05 mm, vias 0 -> 1
- net PWR_3.5_12: track 12.8 -> 19.6 mm, vias 2 -> 5
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