File: Hardware/Schematic v1/Full schematic/Full schematic.kicad_sch (KiCad schematic)
At the start: 301 parts, among them J1 Conn_01x02_Male, J10 Conn_01x01_Male, J2 Reset, J3 Encoder, J4 Failure LED, J5 Bluetooth, J6 Conn_01x02_Male, J7 Display, J8 Buttons, J9 Conn_01x02_Male, K1 G6L-1F-DC5, K2 G6L-1F-DC5, K3 G6L-1F-DC5, K4 G6L-1F-DC5, K5 G6L-1F-DC5, K6 G6L-1F-DC5, Q1 BC847, Q10 IRLML6402, Q11 BC847, Q12 IRFZ44, Q13 BC847, Q14 IRLML6402, Q15 BC847, Q16 BSS138, Q17 BC847, Q18 IRF610, Q19 BC847, Q2 BC847, Q20 IRLML6402, Q21 BC847, Q22 IRLML6402, Q23 BFS17, Q24 AFT05MS003N, Q25 IRLML2502, Q26 IRLML2502, Q27 IRLML2502, Q28 IRLML2502, Q29 IRLML2502, Q3 BC847, Q30 IRLML2502, Q4 BC847, Q5 BC847, Q6 IRLML6402, Q7 IRF4905, Q8 IRLML6402, Q9 IRLML6402, U1 74LVC2T45DC, U10 ICS501, U11 STM32F103C8Tx, U12 CAT24C256, U2 74LVC2T45DC, U3 AD9835, U4 LM27313XMF, U5 LM2734X, U6 LM2734X, U7 MAX1837EUT33-T, U8 UC3843_SOIC8, U9 AD5245BRJZ10, X1 50MHz, Y1 8MHz, Y2 32768Hz

Commit message: - New antenna matcher
- Ready to trace PCB
Parts:
- removed C106: 22uF x 10V, Capacitor_THT:CP_Radial_D4.0mm_P2.00mm, symbol Full-schematic-rescue:CP-Device
- removed C84: 2pF 250V, Capacitor_SMD:C_0805_2012Metric_Pad1.18x1.45mm_HandSolder, symbol Device:C
- removed C86: 62pF 250V, Capacitor_SMD:C_0805_2012Metric_Pad1.18x1.45mm_HandSolder, symbol Device:C
- removed C94: 32pF 250V, Capacitor_SMD:C_0805_2012Metric_Pad1.18x1.45mm_HandSolder, symbol Device:C
- removed J10: Conn_01x01_Male, Connector_PinHeader_2.54mm:PinHeader_1x01_P2.54mm_Vertical, symbol Connector:Conn_01x01_Male
- removed JP3: SWDIO, Connector_PinHeader_2.54mm:PinHeader_1x02_P2.54mm_Vertical, symbol Full-schematic-rescue:Jumper-Device
- removed JP4: SWCLK, Connector_PinHeader_2.54mm:PinHeader_1x02_P2.54mm_Vertical, symbol Full-schematic-rescue:Jumper-Device
- removed K1, K2, K3, K4, K5, K6: G6L-1F-DC5, SamacSys:G6L-1F-DC5, symbol G6L-1F-DC5:G6L-1F-DC5
- removed Q25, Q26, Q27, Q28, Q29, Q30: IRLML2502, Package_TO_SOT_SMD:SOT-23, symbol Device:Q_NMOS_GSD
- removed R91, R95, R96, R97, R98, R99: 100, Resistor_SMD:R_0805_2012Metric_Pad1.20x1.40mm_HandSolder, symbol Device:R
- added C100: 22uF x 10V, Capacitor_THT:CP_Radial_D4.0mm_P2.00mm, symbol Full-schematic-rescue:CP-Device
- added C106: 62pF 250V, Capacitor_SMD:C_0805_2012Metric_Pad1.18x1.45mm_HandSolder, symbol Device:C
- added C107: 2pF 250V, Capacitor_SMD:C_0805_2012Metric_Pad1.18x1.45mm_HandSolder, symbol Device:C
- added C85, C98: 0.1uF, Capacitor_SMD:C_0805_2012Metric_Pad1.18x1.45mm_HandSolder, symbol Device:C
- added J10: Conn_01x03_Male, Connector_PinHeader_2.54mm:PinHeader_1x03_P2.54mm_Vertical, symbol Connector:Conn_01x03_Male
- added K1, K2, K3, K4, K5, K6: IM43TS, Mouser:IM43TS, symbol IM43TS:IM43TS
- added R90: 4.7k, Resistor_SMD:R_0805_2012Metric_Pad1.20x1.40mm_HandSolder, symbol Device:R
- added U12: MCP23017_SS, Package_SO:SSOP-28_5.3x10.2mm_P0.65mm, symbol Interface_Expansion:MCP23017_SS
- C101: value 16pF 250V -> 2pF 250V
- C102: value 8pF 250V -> 16pF 250V
- C104: value 2pF 250V -> 32pF 250V
- C105: value 0.1uF -> 8pF 250V
- L14: footprint Inductor_SMD:L_Pulse_PA4320 -> Mouser:2222SQ301GEC
- renumbered C85 to C84, C87 to C86, C88 to C87, C89 to C88, C90 to C89, C91 to C90, C92 to C91, C93 to C92, C95 to C93, C96 to C94, C97 to C95, C98 to C96, C99 to C97, C100 to C99, R90 to R91, U12 to U13
Connections:
- net ANT_3.5: now also C101.2, C102.2, C103.2, C104.2, C105.2, C106.2, C107.1; no longer C101.1, C102.1, C103.1, C104.1
- net GND: now also C100.2, C85.2, C98.2, J10.1 (Pin_1), K1.3 (COM_1), K2.3 (COM_1), K3.3 (COM_1), K4.3 (COM_1), K5.3 (COM_1), K6.3 (COM_1), U12.10 (VSS), U12.15 (A0), U12.16 (A1), U12.17 (A2); no longer C105.2
- net I2C2_SCL: now also U12.12 (SCK)
- net I2C2_SDA: now also U12.13 (SDA)
- net PWR_3.5_5: now also C100.1, C98.1, R90.1, U12.9 (VDD); no longer C105.1
- net SWCLK: now also J10.2 (Pin_2)
- net SWDIO: now also J10.3 (Pin_3)
- net MATCH_0: no longer names the net of U11.13 (PA3)
- net MATCH_1: no longer names the net of U11.32 (PA11)
- net MATCH_2: no longer names the net of U11.33 (PA12)
- net MATCH_5: no longer names the net of U11.38 (PA15)
- new net: C105.1, K5.4 (NO_1)
- new net: C104.1, K4.4 (NO_1)
- new net: C102.1, K2.4 (NO_1)
- new net: C101.1, K1.4 (NO_1)
- new net: C85.1, R90.2, U12.18 (~{RESET})
- new net: C106.1, C107.2, K6.4 (NO_1)
- new net: C103.1, K3.4 (NO_1)
- new net MATCH0+: K1.1 (COIL+), U12.21 (GPA0)
- new net MATCH0-: K1.8 (COIL-), U12.1 (GPB0)
- new net MATCH1+: K3.1 (COIL+), U12.22 (GPA1)
- new net MATCH1-: K3.8 (COIL-), U12.2 (GPB1)
- new net MATCH2+: K5.1 (COIL+), U12.23 (GPA2)
- new net MATCH2-: K5.8 (COIL-), U12.3 (GPB2)
- new net MATCH3+: K2.1 (COIL+), U12.24 (GPA3)
- new net MATCH3-: K2.8 (COIL-), U12.4 (GPB3)
- new net MATCH4+: K4.1 (COIL+), U12.25 (GPA4)
- new net MATCH4-: K4.8 (COIL-), U12.5 (GPB4)
- new net MATCH5+: K6.1 (COIL+), U12.26 (GPA5)
- new net MATCH5-: K6.8 (COIL-), U12.6 (GPB5)
Other:
- note added: "Address = 20H"
- note added: "Address = 58H"

Commit message: - some schematic fixes
- PCB tracing in progress
Parts:
- added C101, C102, C103, C104, C107, C108, C109, C110, C113, C114, C115, C116: 4.7uF, Capacitor_SMD:C_0805_2012Metric_Pad1.18x1.45mm_HandSolder, symbol Device:C
- added R88: 36k, Resistor_SMD:R_0805_2012Metric_Pad1.20x1.40mm_HandSolder, symbol Device:R
- renumbered C101 to C105, C102 to C106, C103 to C111, C104 to C112, C105 to C117, C106 to C118, C107 to C119, R88 to R89, R89 to R90, R90 to R91, R91 to R92, R92 to R93, R93 to R94, R94 to R95
Connections:
- net MANIP_144: now also R88.1; no longer RV2.1
- net MATCH0+: now also C101.2, C103.2; no longer K1.1 (COIL+)
- net MATCH1+: now also C107.2, C109.2; no longer K3.1 (COIL+)
- net MATCH2+: now also C113.2, C115.2; no longer K5.1 (COIL+)
- net MATCH3+: now also C102.2, C104.2; no longer K2.1 (COIL+)
- net MATCH4+: now also C108.2, C110.2; no longer K4.1 (COIL+)
- net MATCH5+: now also C114.2, C116.2; no longer K6.1 (COIL+)
- new net: R88.2, RV2.1
- new net: C113.1, C115.1, K5.1 (COIL+)
- new net: C108.1, C110.1, K4.1 (COIL+)
- new net: C107.1, C109.1, K3.1 (COIL+)
- new net: C101.1, C103.1, K1.1 (COIL+)
- new net: C114.1, C116.1, K6.1 (COIL+)
- new net: C102.1, C104.1, K2.1 (COIL+)
Other:
- moved on the sheet: C105, C106, C111, C112, C117, C118, C119, K1, K2, K3, K4, K5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

Commit message: PCB tracing in progress
Parts:
- C1: footprint Inductor_SMD:L_0603_1608Metric_Pad1.05x0.95mm_HandSolder -> Capacitor_THT:CP_Radial_D6.3mm_P2.50mm
Changed lines of the file:
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@@
       (effects (font (size 1.27 1.27)) (justify left))
     )
-    (property "Footprint" "Inductor_SMD:L_0603_1608Metric_Pad1.05x0.95mm_HandSolder" (id 2) (at 40.9702 231.14 0)
+    (property "Footprint" "Capacitor_THT:CP_Radial_D6.3mm_P2.50mm" (id 2) (at 40.9702 231.14 0)
       (effects (font (size 1.27 1.27)) hide)
     )
@@
     )
     (path "/00000000-0000-0000-0000-000060da81bd"
-      (reference "C1") (unit 1) (value "100uFx16V") (footprint "Inductor_SMD:L_0603_1608Metric_Pad1.05x0.95mm_HandSolder")
+      (reference "C1") (unit 1) (value "100uFx16V") (footprint "Capacitor_THT:CP_Radial_D6.3mm_P2.50mm")
     )
     (path "/00000000-0000-0000-0000-00005fded36d"
